Commit message: Add LD06 SLAM and Nav2 development

File: ros2_ws/src/pupper_v3_description/description/urdf/pupper_v3.edited.fixed.urdf (robot description, URDF)
Before this commit: robot pupper_v3, 14 links, 13 joints
Links:
- added link lidar_link; collision cylinder length=0.033 radius=0.0195; visual cylinder length=0.033 radius=0.0195
Joints:
- added joint base_link_to_lidar: type fixed, parent base_link, child lidar_link, origin xyz=0.057 0 0.123 rpy=0 0 0
